File: pcb/cybdokey.kicad_sch (KiCad schematic)
At the start: 39 parts, among them J1 USB_A, U1 RP2354_60QFN, U2 MCP1700x-300xxTT, U3 USBLC6-2P6, Y1 ABM8-272-T3

Commit message: started routing
Parts:
- C1, C10, C11, C12, C13, C14, C15, C16, C17, C18, C19, C2, C3, C4, C5, C6, C7, C8, C9: footprint (none) -> Capacitor_SMD:C_0402_1005Metric_Pad0.74x0.62mm_HandSolder
- D1: footprint (none) -> Diode_SMD:D_SOD-323F
- J1: footprint Connector_USB:USB_A_CNCTech_1001-011-01101_Horizontal -> PCM_Connector_USB_PCB_Edge:USB_A_PCB_Edge_receptacle
- L1: footprint (none) -> imports:INDC1608X95N
- R1, R2, R3, R4, R5, R6, R7, R8, R9: footprint (none) -> Resistor_SMD:R_0402_1005Metric_Pad0.72x0.64mm_HandSolder
- TP1: footprint (none) -> imports:touchpad
Connections:
- net USB_D-: now reaches J1.2 (D-), U3.3 (I/O2)
- net USB_D+: now reaches J1.3 (D+), U3.1 (I/O1)
- net USB_DM renamed PROT_USB_D-
- net USB_DP renamed PROT_USB_D+
Changed lines of the file:
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@@
 	(wire
 		(pts
-			(xy 71.12 36.83) (xy 60.96 36.83)
+			(xy 76.2 36.83) (xy 60.96 36.83)
 		)
 		(stroke
@@
 	(wire
 		(pts
-			(xy 71.12 39.37) (xy 60.96 39.37)
+			(xy 76.2 39.37) (xy 60.96 39.37)
 		)
 		(stroke
@@
 		)
 	)
-	(label "USB_DP"
-		(at 71.12 36.83 180)
+	(label "USB_D-"
+		(at 49.53 39.37 180)
 		(effects
 			(font
@@
 		)
 	)
-	(label "USB_DM"
-		(at 71.12 39.37 180)
+	(label "PROT_USB_D+"
+		(at 76.2 36.83 180)
+		(effects
+			(font
+				(size 1.27 1.27)
+			)
+			(justify right bottom)
+		)
+	)
+	(label "PROT_USB_D-"
+		(at 76.2 39.37 180)
 		(effects
 			(font
@@
 		)
 	)
-	(label "USB_DP"
+	(label "PROT_USB_D+"
 		(at 191.77 92.71 180)
 		(effects
@@
 		)
 	)
-	(label "USB_DM"
+	(label "PROT_USB_D-"
 		(at 191.77 95.25 180)
 		(effects
@@
 		)
 	)
+	(label "USB_D+"
+		(at 49.53 36.83 180)
+		(effects
+			(font
+				(size 1.27 1.27)
+			)
+			(justify right bottom)
+		)
+	)
 	(label "QSPI_SS"
 		(at 227.33 30.48 0)
@@
 			)
 		)
-		(property "Footprint" ""
+		(property "Footprint" "Resistor_SMD:R_0402_1005Metric_Pad0.72x0.64mm_HandSolder"
 			(at 170.18 97.028 90)
 			(effects
@@
 			)
 		)
-		(property "Footprint" ""
+		(property "Footprint" "Capacitor_SMD:C_0402_1005Metric_Pad0.74x0.62mm_HandSolder"
 			(at 130.5052 39.37 0)
 			(effects
@@
 			)
 		)
-		(property "Footprint" ""
+		(property "Footprint" "Capacitor_SMD:C_0402_1005Metric_Pad0.74x0.62mm_HandSolder"
 			(at 167.64 25.7048 0)
 			(effects
@@
 			)
 		)
-		(property "Footprint" "Connector_USB:USB_A_CNCTech_1001-011-01101_Horizontal"
+		(property "Footprint" "PCM_Connector_USB_PCB_Edge:USB_A_PCB_Edge_receptacle"
 			(at 36.83 38.1 0)
 			(effects
@@
 			)
 		)
-		(property "Footprint" ""
+		(property "Footprint" "Capacitor_SMD:C_0402_1005Metric_Pad0.74x0.62mm_HandSolder"
 			(at 83.5152 72.39 0)
 			(effects
@@
 			)
 		)
-		(property "Footprint" ""
+		(property "Footprint" "Capacitor_SMD:C_0402_1005Metric_Pad0.74x0.62mm_HandSolder"
 			(at 225.7552 73.66 0)
 			(effects
@@
 			)
 		)
-		(property "Footprint" ""
+		(property "Footprint" "Capacitor_SMD:C_0402_1005Metric_Pad0.74x0.62mm_HandSolder"
 			(at 80.9752 93.98 0)
 			(effects
@@
 			)
 		)
-		(property "Footprint" ""
+		(property "Footprint" "Capacitor_SMD:C_0402_1005Metric_Pad0.74x0.62mm_HandSolder"
 			(at 202.8952 73.66 0)
 			(effects
@@
 			)
 		)
-		(property "Footprint" ""
+		(property "Footprint" "Capacitor_SMD:C_0402_1005Metric_Pad0.74x0.62mm_HandSolder"
 			(at 180.0352 73.66 0)
 			(effects
@@
 			)
 		)
-		(property "Footprint" ""
+		(property "Footprint" "Resistor_SMD:R_0402_1005Metric_Pad0.72x0.64mm_HandSolder"
 			(at 198.12 38.608 90)
 			(effects
@@
 			)
 		)
-		(property "Footprint" ""
+		(property "Footprint" "Resistor_SMD:R_0402_1005Metric_Pad0.72x0.64mm_HandSolder"
 			(at 234.95 117.602 90)
 			(effects
@@
 			)
 		)
-		(property "Footprint" ""
+		(property "Footprint" "Capacitor_SMD:C_0402_1005Metric_Pad0.74x0.62mm_HandSolder"
 			(at 168.6052 73.66 0)
 			(effects
@@
 			)
 		)
-		(property "Footprint" ""
+		(property "Footprint" "Capacitor_SMD:C_0402_1005Metric_Pad0.74x0.62mm_HandSolder"
 			(at 160.02 37.7952 0)
 			(effects
@@
 			)
 		)
-		(property "Footprint" ""
+		(property "Footprint" "Resistor_SMD:R_0402_1005Metric_Pad0.72x0.64mm_HandSolder"
 			(at 170.18 94.488 90)
 			(effects
@@
 			)
 		)
-		(property "Footprint" ""
+		(property "Footprint" "imports:INDC1608X95N"
 			(at 58.42 99.06 0)
 			(effects
@@
 			)
 		)
-		(property "Footprint" ""
+		(property "Footprint" "Capacitor_SMD:C_0402_1005Metric_Pad0.74x0.62mm_HandSolder"
 			(at 103.8352 39.37 0)
 			(effects
@@
 			)
 		)
-		(property "Footprint" ""
+		(property "Footprint" "Resistor_SMD:R_0402_1005Metric_Pad0.72x0.64mm_HandSolder"
 			(at 245.618 25.4 90)
 			(effects
@@
 			)
 		)
-		(property "Footprint" ""
+		(property "Footprint" "Resistor_SMD:R_0402_1005Metric_Pad0.72x0.64mm_HandSolder"
 			(at 245.618 44.45 90)
 			(effects
@@
 			)
 		)
-		(property "Footprint" ""
+		(property "Footprint" "Diode_SMD:D_SOD-323F"
 			(at 77.47 30.48 0)
 			(effects
@@
 			)
 		)
-		(property "Footprint" ""
+		(property "Footprint" "Resistor_SMD:R_0402_1005Metric_Pad0.72x0.64mm_HandSolder"
 			(at 74.93 86.868 90)
 			(effects
@@
 			)
 		)
-		(property "Footprint" ""
+		(property "Footprint" "Capacitor_SMD:C_0402_1005Metric_Pad0.74x0.62mm_HandSolder"
 			(at 157.1752 73.66 0)
 			(effects
@@
 			)
 		)
-		(property "Footprint" ""
+		(property "Footprint" "Capacitor_SMD:C_0402_1005Metric_Pad0.74x0.62mm_HandSolder"
 			(at 32.7152 104.14 0)
 			(effects
@@
 			)
 		)
-		(property "Footprint" ""
+		(property "Footprint" "Capacitor_SMD:C_0402_1005Metric_Pad0.74x0.62mm_HandSolder"
 			(at 72.0852 72.39 0)
 			(effects
@@
 			)
 		)
-		(property "Footprint" ""
+		(property "Footprint" "Capacitor_SMD:C_0402_1005Metric_Pad0.74x0.62mm_HandSolder"
 			(at 214.3252 73.66 0)
 			(effects
@@
 			)
 		)
-		(property "Footprint" ""
+		(property "Footprint" "imports:touchpad"
 			(at 246.38 124.46 0)
 			(effects
@@
 			)
 		)
-		(property "Footprint" ""
+		(property "Footprint" "Capacitor_SMD:C_0402_1005Metric_Pad0.74x0.62mm_HandSolder"
 			(at 191.4652 73.66 0)
 			(effects
@@
 			)
 		)
-		(property "Footprint" ""
+		(property "Footprint" "Resistor_SMD:R_0402_1005Metric_Pad0.72x0.64mm_HandSolder"
 			(at 32.258 185.42 90)
 			(effects
@@
 			)
 		)
-		(property "Footprint" ""
+		(property "Footprint" "Capacitor_SMD:C_0402_1005Metric_Pad0.74x0.62mm_HandSolder"
 			(at 47.9552 104.14 0)
 			(effects
@@
 			)
 		)
-		(property "Footprint" ""
+		(property "Footprint" "Resistor_SMD:R_0402_1005Metric_Pad0.72x0.64mm_HandSolder"
 			(at 32.258 166.37 90)
 			(effects
@@
 			)
 		)
-		(property "Footprint" ""
+		(property "Footprint" "Capacitor_SMD:C_0402_1005Metric_Pad0.74x0.62mm_HandSolder"
 			(at 248.6152 73.66 0)
 			(effects
@@
 			)
 		)
-		(property "Footprint" ""
+		(property "Footprint" "Capacitor_SMD:C_0402_1005Metric_Pad0.74x0.62mm_HandSolder"
 			(at 237.1852 73.66 0)
 			(effects
@@
 			)
 		)
-		(property "Footprint" ""
+		(property "Footprint" "Capacitor_SMD:C_0402_1005Metric_Pad0.74x0.62mm_HandSolder"
 			(at 60.6552 72.39 0)
 			(effects

Commit message: more routing
Parts:
- removed C14: 100nF, Capacitor_SMD:C_0402_1005Metric_Pad0.74x0.62mm_HandSolder, symbol Device:C
- removed JP2: SolderJumper_2_Open, Jumper:SolderJumper-2_P1.3mm_Open_TrianglePad1.0x1.5mm, symbol Jumper:SolderJumper_2_Open
- removed R8: 10kR, Resistor_SMD:R_0402_1005Metric_Pad0.72x0.64mm_HandSolder, symbol Device:R
- removed R9: 1kR, Resistor_SMD:R_0402_1005Metric_Pad0.72x0.64mm_HandSolder, symbol Device:R
- added TP2: run, TestPoint:TestPoint_Pad_1.0x1.0mm, symbol Connector:TestPoint
- added TP3: 3V3, TestPoint:TestPoint_Pad_1.0x1.0mm, symbol Connector:TestPoint
- added TP4: GND, TestPoint:TestPoint_Pad_1.0x1.0mm, symbol Connector:TestPoint
Connections:
- net +3V3: now also TP3.1
- net GND: now also TP4.1
- net PROT_USB_D+: now also U3.4 (I/O2); no longer U3.6 (I/O1)
- net PROT_USB_D-: now also U3.6 (I/O1); no longer U3.4 (I/O2)
- net USB_D+: now also U3.3 (I/O2); no longer U3.1 (I/O1)
- net USB_D-: now also U3.1 (I/O1); no longer U3.3 (I/O2)
- net RUN: no longer names the net of U1.26 (RUN)
- net RUN: now also TP2.1
Other:
- note removed: "Reset"
- moved on the sheet: U3

Commit message: routing done... for now
Parts:
- removed C13: 100nF, Capacitor_SMD:C_0402_1005Metric_Pad0.74x0.62mm_HandSolder, symbol Device:C
Connections:
- net TOUCH_BTN: now also U1.15 (GPIO11); no longer U1.17 (GPIO13)
- no-connect marks 36 -> 35
Changed lines of the file:
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@@
 	)
 	(junction
-		(at 224.79 64.77)
-		(diameter 0)
-		(color 0 0 0 0)
-	)
-	(junction
 		(at 71.12 30.48)
 		(diameter 0)
@@
 	)
 	(junction
-		(at 236.22 74.93)
-		(diameter 0)
-		(color 0 0 0 0)
-	)
-	(junction
 		(at 179.07 64.77)
 		(diameter 0)
@@
 	)
 	(no_connect
-		(at 154.94 130.81)
-	)
-	(no_connect
 		(at 154.94 128.27)
 	)
@@
 	(wire
 		(pts
+			(xy 154.94 130.81) (xy 167.64 130.81)
+		)
+		(stroke
+			(width 0)
+			(type default)
+		)
+	)
+	(wire
+		(pts
 			(xy 46.99 92.71) (xy 46.99 93.98)
 		)
@@
 	(wire
 		(pts
-			(xy 224.79 74.93) (xy 236.22 74.93)
-		)
-		(stroke
-			(width 0)
-			(type default)
-		)
-	)
-	(wire
-		(pts
 			(xy 179.07 74.93) (xy 190.5 74.93)
 		)
@@
 	(wire
 		(pts
-			(xy 236.22 66.04) (xy 236.22 64.77)
-		)
-		(stroke
-			(width 0)
-			(type default)
-		)
-	)
-	(wire
-		(pts
 			(xy 139.7 83.82) (xy 139.7 85.09)
 		)
@@
 	(wire
 		(pts
-			(xy 224.79 64.77) (xy 236.22 64.77)
-		)
-		(stroke
-			(width 0)
-			(type default)
-		)
-	)
-	(wire
-		(pts
 			(xy 64.77 101.6) (xy 64.77 93.98)
 		)
@@
 	(wire
 		(pts
-			(xy 236.22 73.66) (xy 236.22 74.93)
-		)
-		(stroke
-			(width 0)
-			(type default)
-		)
-	)
-	(wire
-		(pts
 			(xy 215.9 119.38) (xy 231.14 119.38)
 		)
@@
 	(wire
 		(pts
-			(xy 236.22 76.2) (xy 236.22 74.93)
+			(xy 224.79 76.2) (xy 224.79 74.93)
 		)
 		(stroke
@@
 	(wire
 		(pts
-			(xy 154.94 135.89) (xy 167.64 135.89)
-		)
-		(stroke
-			(width 0)
-			(type default)
-		)
-	)
-	(wire
-		(pts
 			(xy 113.03 83.82) (xy 119.38 83.82)
 		)
@@
 		)
 	)
-	(label "TOUCH_BTN"
-		(at 167.64 135.89 180)
-		(effects
-			(font
-				(size 1.27 1.27)
-			)
-			(justify right bottom)
-		)
-	)
 	(label "PROT_USB_D-"
 		(at 191.77 95.25 180)
@@
 		)
 	)
+	(label "TOUCH_BTN"
+		(at 167.64 130.81 180)
+		(effects
+			(font
+				(size 1.27 1.27)
+			)
+			(justify right bottom)
+		)
+	)
 	(label "XIN"
 		(at 212.09 26.67 180)
@@
 	(symbol
 		(lib_id "power:GND")
-		(at 236.22 76.2 0)
+		(at 224.79 76.2 0)
 		(unit 1)
 		(exclude_from_sim no)
@@
 		(fields_autoplaced yes)
 		(property "Reference" "#PWR012"
-			(at 236.22 82.55 0)
+			(at 224.79 82.55 0)
 			(effects
 				(font
@@
 		)
 		(property "Value" "GND"
-			(at 236.22 81.28 0)
+			(at 224.79 81.28 0)
 			(effects
 				(font
@@
 		)
 		(property "Footprint" ""
-			(at 236.22 76.2 0)
+			(at 224.79 76.2 0)
 			(effects
 				(font
@@
 		)
 		(property "Datasheet" ""
-			(at 236.22 76.2 0)
+			(at 224.79 76.2 0)
 			(effects
 				(font
@@
 		)
 		(property "Description" "Power symbol creates a global label with name \"GND\" , ground"
-			(at 236.22 76.2 0)
+			(at 224.79 76.2 0)
 			(effects
 				(font
@@
 					(unit 1)
 				)
-			)
-		)
-	)
-	(symbol
-		(lib_id "Device:C")
-		(at 236.22 69.85 0)
-		(unit 1)
-		(exclude_from_sim no)
-		(in_bom yes)
-		(on_board yes)
-		(dnp no)
-		(property "Reference" "C13"
-			(at 238.76 68.58 0)
-			(effects
-				(font
-					(size 1.27 1.27)
-				)
-				(justify left)
-			)
-		)
-		(property "Value" "100nF"
-			(at 238.76 71.12 0)
-			(effects
-				(font
-					(size 1.27 1.27)
-				)
-				(justify left)
-			)
-		)
-		(property "Footprint" "Capacitor_SMD:C_0402_1005Metric_Pad0.74x0.62mm_HandSolder"
-			(at 237.1852 73.66 0)
-			(effects
-				(font
-					(size 1.27 1.27)
-				)
-				(hide yes)
-			)
-		)
-		(property "Datasheet" "~"
-			(at 236.22 69.85 0)
-			(effects
-				(font
-					(size 1.27 1.27)
-				)
-				(hide yes)
-			)
-		)
-		(property "Description" "Unpolarized capacitor"
-			(at 236.22 69.85 0)
-			(effects
-				(font
-					(size 1.27 1.27)
-				)
-				(hide yes)
-			)
-		)
-		(pin "1"
-		)
-		(pin "2"
-		)
-		(instances
-			(project "cybdokey"
-				(path "/5a6e220c-1a09-4082-aaa1-5a3866ea77ed"
-					(reference "C13")
-					(unit 1)
-				)

Commit message: cleaned up routing
Parts:
- D2: footprint LED_SMD:LED_WS2812B_PLCC4_5.0x5.0mm_P3.2mm -> imports:SK6812MINI-E_fixed
Changed lines of the file:
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@@
 			)
 		)
-		(property "Footprint" "LED_SMD:LED_WS2812B_PLCC4_5.0x5.0mm_P3.2mm"
+		(property "Footprint" "imports:SK6812MINI-E_fixed"
 			(at 236.22 152.4 0)
 			(effects

Commit message: changed LED, moving back to windows
Parts:
- removed D2: WS2812B, imports:SK6812MINI-E_fixed, symbol LED:WS2812B
- added D3: LED_RKBG, LED_SMD:LED_Kingbright_AAA3528ESGCT, symbol Device:LED_RKBG
Connections:
- net GND: now also D3.2 (K)
- net LED_R: now reaches U1.18 (GPIO14)
- net LED_R: now also D3.1 (RA)
- net LED_B: now reaches U1.4 (GPIO2)
- net LED_B: now also D3.3 (BA)
- net LED renamed LED_G
- net LED_G: now also D3.4 (GA)
- no-connect marks 35 -> 32

Commit message: add new touch button footprint and add some branding
Parts:
- added R8, R9: 220R, Resistor_SMD:R_0402_1005Metric_Pad0.72x0.64mm_HandSolder, symbol Device:R
- D3: footprint LED_SMD:LED_Kingbright_AAA3528ESGCT -> imports:LED-SMD_4P-L3.2-W2.8_XZMDKCBDDG45S-9
Connections:
- net LED_B: now also R8.2; no longer D3.3 (BA), U1.4 (GPIO2)
- net LED_G: no longer D3.4 (GA)
- net LED_R: now also R9.1; no longer D3.1 (RA)
- new net: D3.3 (BA), R8.1
- new net: D3.1 (RA), R9.2
- no-connect marks 32 -> 35
Changed lines of the file:
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@@
 	)
 	(no_connect
+		(at 154.94 113.03)
+	)
+	(no_connect
 		(at 154.94 118.11)
 	)
@@
 	)
 	(no_connect
+		(at 154.94 107.95)
+	)
+	(no_connect
 		(at 91.44 167.64)
 	)
@@
 	)
 	(no_connect
+		(at 198.12 138.43)
+	)
+	(no_connect
 		(at 154.94 140.97)
 	)
@@
 	(wire
 		(pts
-			(xy 190.5 143.51) (xy 198.12 143.51)
+			(xy 180.34 143.51) (xy 189.23 143.51)
 		)
 		(stroke
@@
 	(wire
 		(pts
-			(xy 190.5 138.43) (xy 198.12 138.43)
+			(xy 180.34 133.35) (xy 189.23 133.35)
 		)
 		(stroke
@@
 	(wire
 		(pts
-			(xy 154.94 107.95) (xy 166.37 107.95)
-		)
-		(stroke
-			(width 0)
-			(type default)
-		)
-	)
-	(wire
-		(pts
 			(xy 88.9 96.52) (xy 91.44 96.52)
 		)
@@
 	(wire
 		(pts
-			(xy 190.5 133.35) (xy 198.12 133.35)
-		)
-		(stroke
-			(width 0)
-			(type default)
-		)
-	)
-	(wire
-		(pts
 			(xy 49.53 30.48) (xy 71.12 30.48)
 		)
@@
 	(wire
 		(pts
+			(xy 196.85 133.35) (xy 198.12 133.35)
+		)
+		(stroke
+			(width 0)
+			(type default)
+		)
+	)
+	(wire
+		(pts
 			(xy 31.75 106.68) (xy 31.75 107.95)
 		)
@@
 	(wire
 		(pts
+			(xy 196.85 143.51) (xy 198.12 143.51)
+		)
+		(stroke
+			(width 0)
+			(type default)
+		)
+	)
+	(wire
+		(pts
 			(xy 243.84 20.32) (xy 243.84 21.59)
 		)
@@
 	)
 	(label "LED_R"
-		(at 190.5 143.51 0)
+		(at 180.34 143.51 0)
 		(effects
 			(font
@@
 		)
 	)
-	(label "LED_B"
-		(at 190.5 133.35 0)
-		(effects
-			(font
-				(size 1.27 1.27)
-			)
-			(justify left bottom)
-		)
-	)
 	(label "QSPI_SS"
 		(at 82.55 114.3 0)
@@
 		)
 	)
-	(label "LED_B"
-		(at 166.37 107.95 180)
-		(effects
-			(font
-				(size 1.27 1.27)
-			)
-			(justify right bottom)
-		)
-	)
 	(label "USB_D+"
 		(at 49.53 36.83 180)
@@
 		)
 	)
-	(label "LED_G"
-		(at 190.5 138.43 0)
+	(label "LED_B"
+		(at 180.34 133.35 0)
 		(effects
 			(font
@@
 	)
 	(symbol
+		(lib_id "Device:R")
+		(at 193.04 133.35 270)
+		(unit 1)
+		(exclude_from_sim no)
+		(in_bom yes)
+		(on_board yes)
+		(dnp no)
+		(property "Reference" "R8"
+			(at 193.04 129.54 90)
+			(effects
+				(font
+					(size 1.27 1.27)
+				)
+			)
+		)
+		(property "Value" "220R"
+			(at 193.04 127 90)
+			(effects
+				(font
+					(size 1.27 1.27)
+				)
+			)
+		)
+		(property "Footprint" "Resistor_SMD:R_0402_1005Metric_Pad0.72x0.64mm_HandSolder"
+			(at 193.04 131.572 90)
+			(effects
+				(font
+					(size 1.27 1.27)
+				)
+				(hide yes)
+			)
+		)
+		(property "Datasheet" "~"
+			(at 193.04 133.35 0)
+			(effects
+				(font
+					(size 1.27 1.27)
+				)
+				(hide yes)
+			)
+		)
+		(property "Description" "Resistor"
+			(at 193.04 133.35 0)
+			(effects
+				(font
+					(size 1.27 1.27)
+				)
+				(hide yes)
+			)
+		)
+		(pin "2"
+		)
+		(pin "1"
+		)
+		(instances
+			(project "cybdokey"
+				(path "/5a6e220c-1a09-4082-aaa1-5a3866ea77ed"
+					(reference "R8")
+					(unit 1)
+				)
+			)
+		)
+	)
+	(symbol
 		(lib_id "power:GND")
 		(at 80.01 95.25 0)
@@
 			)
 		)
-		(property "Footprint" "LED_SMD:LED_Kingbright_AAA3528ESGCT"
+		(property "Footprint" "imports:LED-SMD_4P-L3.2-W2.8_XZMDKCBDDG45S-9"
 			(at 203.2 137.16 0)
 			(effects
@@
 					(unit 1)
 				)
+			)
+		)
+	)
+	(symbol
+		(lib_id "Device:R")
+		(at 193.04 143.51 90)
+		(unit 1)
+		(exclude_from_sim no)
+		(in_bom yes)
+		(on_board yes)
+		(dnp no)
+		(property "Reference" "R9"
+			(at 193.04 147.32 90)
+			(effects
+				(font
+					(size 1.27 1.27)
+				)
+			)
+		)
+		(property "Value" "220R"
+			(at 193.04 149.86 90)
+			(effects
+				(font
+					(size 1.27 1.27)
+				)
+			)
+		)
+		(property "Footprint" "Resistor_SMD:R_0402_1005Metric_Pad0.72x0.64mm_HandSolder"
+			(at 193.04 145.288 90)
+			(effects
+				(font
+					(size 1.27 1.27)
+				)
+				(hide yes)
+			)
+		)
+		(property "Datasheet" "~"
+			(at 193.04 143.51 0)
+			(effects
+				(font
+					(size 1.27 1.27)
+				)
+				(hide yes)
+			)
+		)
+		(property "Description" "Resistor"
+			(at 193.04 143.51 0)
+			(effects
+				(font
+					(size 1.27 1.27)
+				)
+				(hide yes)
+			)
+		)
+		(pin "2"
+		)
+		(pin "1"
+		)
+		(instances
+			(project "cybdokey"
+				(path "/5a6e220c-1a09-4082-aaa1-5a3866ea77ed"
+					(reference "R9")
+					(unit 1)
+				)

Commit message: polishing, started with some renders
Parts:
- C18, C19: value 4.7uF -> 15pF
Connections:
- net LED_G is gone; now on net LED_B: U1.16 (GPIO12)
Changed lines of the file:
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@@
 		)
 	)
-	(label "LED_G"
+	(label "LED_B"
 		(at 167.64 133.35 180)
 		(effects
@@
 			)
 		)
-		(property "Value" "4.7uF"
+		(property "Value" "15pF"
 			(at 163.83 21.59 90)
 			(effects
@@
 			)
 		)
-		(property "Value" "4.7uF"
+		(property "Value" "15pF"
 			(at 163.83 42.926 90)
 			(effects
