File: pcb/cybdokey.kicad_pcb (KiCad board)
At the start: 2 copper layers, 12 x 32 mm, 41 parts, among them J1 USB_A, U1 RP2354_60QFN, U2 MCP1700x-300xxTT, U3 USBLC6-2P6, Y1 ABM8-272-T3

Commit message: render stuff, add zine page
Routing:
- net +3V3: track 87.3 -> 84.1 mm, vias 13 -> 12
